Commit message: update for passive joints

File: resources/robots/go1_aw/urdf/go1_aw.urdf (robot description, URDF)
Before this commit: robot go1_fw_description, 27 links, 26 joints
Joints:
- joint FR_roller_foot_joint: axis 0 1 0 -> 0 0 1; origin xyz=0 0 0 rpy=0 0 0 -> xyz=0 0 0 rpy=1.57 0 0
- joint RL_roller_foot_joint: axis 0 1 0 -> 0 0 1; origin xyz=0 0 0 rpy=0 0 0 -> xyz=0 0 0 rpy=-1.57 0 0.3
- joint RR_roller_foot_joint: axis 0 1 0 -> 0 0 1; origin xyz=0 0 0 rpy=0 0 0 -> xyz=0 0 0 rpy=1.57 0 -0.3
