Commit message: update scripts

File: resources/robots/go1_fw/urdf/go1_fw.urdf (robot description, URDF)
Before this commit: robot go1_fw_description, 25 links, 24 joints
Links:
- link FL_roller_foot: geometry collision mesh filename=../meshes/wheel_tire.stl scale=0.5 0.5 0.5; visual mesh filename=../meshes/wheel_tire.stl scale=0.5 0.5 0.5
- link FR_roller_foot: geometry collision mesh filename=../meshes/wheel_tire.stl scale=0.5 0.5 0.5; visual mesh filename=../meshes/wheel_tire.stl scale=0.5 0.5 0.5
Joints:
- joint FL_roller_foot_joint: origin xyz=0 0.04 0 rpy=0 0 0 -> xyz=-0.025 -0.00 -0.04 rpy=0 0 0
- joint FR_roller_foot_joint: origin xyz=0 -0.04 0 rpy=0 0 0 -> xyz=-0.025 -0.00 -0.04 rpy=0 0 0
