Commit message: uprate

File: resources/robots/go1_fw/urdf/go1_fw3.urdf (robot description, URDF)
Before this commit: robot go1_fw_description, 25 links, 24 joints
Links:
- link FL_ankle: geometry collision box size=0.04 0.07 0.01; collision sphere radius=0.02
- link FL_roller_foot: geometry collision mesh filename=../meshes/wheel_tire.stl scale=0.5 0.5 0.2; visual mesh filename=../meshes/wheel_tire.stl scale=0.5 0.5 0.4
- link FR_ankle: geometry collision box size=0.04 0.07 0.01; collision sphere radius=0.02
- link FR_roller_foot: geometry collision mesh filename=../meshes/wheel_tire.stl scale=0.5 0.5 0.2; visual mesh filename=../meshes/wheel_tire.stl scale=0.5 0.5 0.4
