Commit message: wheel with angle

File: resources/robots/go1_fw/urdf/go1_fw3_contact_new.urdf (robot description, URDF)
Before this commit: robot go1_fw_description, 25 links, 24 joints
Joints:
- joint FL_roller_foot_joint: origin xyz=0 0 0 rpy=-1.57 0 0.1 -> xyz=-0.022 0 -0.05 rpy=-1.57 0 0.4
- joint FR_roller_foot_joint: origin xyz=0 0 0 rpy=1.57 0 -0.1 -> xyz=-0.022 0 -0.05 rpy=1.57 0 -0.4

Commit message: wheel with angle

File: resources/robots/go1_fw/urdf/go1_fw3_contact_new.urdf (robot description, URDF)
Before this commit: robot go1_fw_description, 25 links, 24 joints
Joints:
- joint FL_roller_foot_joint: origin xyz=-0.022 0 -0.05 rpy=-1.57 0 0.4 -> xyz=-0.022 0 -0.05 rpy=-1.57 0 0.1
- joint FR_roller_foot_joint: origin xyz=-0.022 0 -0.05 rpy=1.57 0 -0.4 -> xyz=-0.022 0 -0.05 rpy=1.57 0 -0.1

Commit message: Your commit message

File: resources/robots/go1_fw/urdf/go1_fw3_contact_new.urdf (robot description, URDF)
Before this commit: robot go1_fw_description, 25 links, 24 joints
Joints:
- joint FL_roller_foot_joint: origin xyz=-0.022 0 -0.05 rpy=-1.57 0 0.1 -> xyz=-0.022 0 -0.05 rpy=-1.57 0 0
- joint FR_roller_foot_joint: origin xyz=-0.022 0 -0.05 rpy=1.57 0 -0.1 -> xyz=-0.022 0 -0.05 rpy=1.57 0 0

Commit message: remove footclearence

File: resources/robots/go1_fw/urdf/go1_fw3_contact_new.urdf (robot description, URDF)
Before this commit: robot go1_fw_description, 25 links, 24 joints
Joints:
- joint FL_roller_foot_joint: origin xyz=-0.022 0 -0.05 rpy=-1.57 0 0 -> xyz=-0.025 0 -0.04 rpy=-1.57 0 -0.1
- joint FR_roller_foot_joint: origin xyz=-0.022 0 -0.05 rpy=1.57 0 0 -> xyz=-0.025 0 -0.04 rpy=1.57 0 0.1
