Commit message: add tilt wheel env

File: resources/robots/go1_fw/urdf/go1_fw3_wheel_tilt.urdf (robot description, URDF)
Before this commit: robot go1_fw_description, 27 links, 26 joints
Links:
- removed link FL_turn
- removed link FR_turn
- added link FL_tilt
- added link FR_tilt
Joints:
- removed joint FL_turn_joint
- removed joint FR_turn_joint
- added joint FL_tilt_joint: type fixed, parent FL_ankle, child FL_tilt, origin xyz=-0.035 -0.00 -0.035 rpy=0 -0.8 0
- added joint FR_tilt_joint: type fixed, parent FR_ankle, child FR_tilt, origin xyz=-0.035 -0.00 -0.035 rpy=0 -0.8 0
- joint FL_roller_foot_joint: parent FL_turn -> FL_tilt
- joint FR_roller_foot_joint: parent FR_turn -> FR_tilt
