Commit message: add tilt urdf

File: resources/robots/go1_fw/urdf/go1_fw3_contact_turning_wheel.urdf (robot description, URDF)
Before this commit: robot go1_fw_description, 27 links, 26 joints
Links:
- removed link FL_tilt
- removed link FR_tilt
- added link FL_turn
- added link FR_turn
Joints:
- removed joint FL_tilt_joint
- removed joint FR_tilt_joint
- added joint FL_turn_joint: type revolute, parent FL_ankle, child FL_turn, origin xyz=-0.035 -0.00 -0.035 rpy=0 -0.8 0, axis 1 0 0, limit lower=-1.57 upper=1.57 effort=33.5 velocity=28
- added joint FR_turn_joint: type revolute, parent FR_ankle, child FR_turn, origin xyz=-0.035 -0.00 -0.035 rpy=0 -0.8 0, axis 1 0 0, limit lower=-1.57 upper=1.57 effort=33.5 velocity=28
- joint FL_roller_foot_joint: parent FL_tilt -> FL_turn
- joint FR_roller_foot_joint: parent FR_tilt -> FR_turn
