Commit message: update wheel urdf

File: resources/robots/go1_fw/urdf/go1_fw3_contact.urdf (robot description, URDF)
Before this commit: robot go1_fw_description, 27 links, 26 joints
Links:
- removed link FL_contact
- removed link FR_contact
- link FL_roller_foot: geometry collision sphere radius=0.03; visual mesh filename=../meshes/wheel_tire.stl scale=0.5 0.5 0.4
- link FR_roller_foot: geometry collision sphere radius=0.03; visual mesh filename=../meshes/wheel_tire.stl scale=0.5 0.5 0.4
Joints:
- removed joint FL_contact_joint
- removed joint FR_contact_joint

Commit message: update

File: resources/robots/go1_fw/urdf/go1_fw3_contact.urdf (robot description, URDF)
Before this commit: robot go1_fw_description, 25 links, 24 joints
Joints:
- joint FL_roller_foot_joint: axis 0 1 0 -> -0 1 0

Commit message: update urdf

File: resources/robots/go1_fw/urdf/go1_fw3_contact.urdf (robot description, URDF)
Before this commit: robot go1_fw_description, 25 links, 24 joints
Links:
- link FL_ankle: geometry collision sphere radius=0.02; visual mesh filename=../meshes/hunong.stl scale=0.1 0.1 0.1
- link FR_ankle: geometry collision sphere radius=0.02; visual mesh filename=../meshes/hunong.stl scale=0.1 0.1 0.1

Commit message: update 0 speed

File: resources/robots/go1_fw/urdf/go1_fw3_contact.urdf (robot description, URDF)
Before this commit: robot go1_fw_description, 25 links, 24 joints
Links:
- link FL_ankle: geometry collision box size=0.04 0.07 0.01; collision sphere radius=0.02
- link FR_ankle: geometry collision box size=0.04 0.07 0.01; collision sphere radius=0.02
