Commit message: env for tilt angle

File: resources/robots/go1_fw/urdf/go1_fw3_contact_tilt_wheel.urdf (robot description, URDF)
Before this commit: robot go1_fw_description, 27 links, 26 joints
Joints:
- removed joint FL_turn_joint
- removed joint FR_turn_joint
- added joint FL_tilt_joint: type revolute, parent FL_ankle, child FL_turn, origin xyz=-0.035 -0.00 -0.035 rpy=0 -0.8 0, axis 1 0 0, limit lower=-0.01 upper=0.01 effort=33.5 velocity=28
- added joint FR_tilt_joint: type revolute, parent FR_ankle, child FR_turn, origin xyz=-0.035 -0.00 -0.035 rpy=0 -0.8 0, axis 1 0 0, limit lower=-0.01 upper=-0.01 effort=33.5 velocity=28

Commit message: update tilt env

File: resources/robots/go1_fw/urdf/go1_fw3_contact_tilt_wheel.urdf (robot description, URDF)
Before this commit: robot go1_fw_description, 27 links, 26 joints
Links:
- removed link FL_turn
- removed link FR_turn
- added link FL_tilt
- added link FR_tilt
Joints:
- joint FL_roller_foot_joint: parent FL_turn -> FL_tilt
- joint FL_tilt_joint: child FL_turn -> FL_tilt
- joint FR_roller_foot_joint: parent FR_turn -> FR_tilt
- joint FR_tilt_joint: child FR_turn -> FR_tilt

Commit message: update tilt setup

File: resources/robots/go1_fw/urdf/go1_fw3_contact_tilt_wheel.urdf (robot description, URDF)
Before this commit: robot go1_fw_description, 27 links, 26 joints
Joints:
- joint FL_tilt_joint: limit lower=-0.01 upper=0.01 effort=33.5 velocity=28 -> lower=-0.01 upper=0.01 effort=0 velocity=100
- joint FR_tilt_joint: limit lower=-0.01 upper=-0.01 effort=33.5 velocity=28 -> lower=-0.01 upper=-0.01 effort=0 velocity=100

Commit message: update tilt

File: resources/robots/go1_fw/urdf/go1_fw3_contact_tilt_wheel.urdf (robot description, URDF)
Before this commit: robot go1_fw_description, 27 links, 26 joints
Joints:
- joint FL_tilt_joint: limit lower=-0.01 upper=0.01 effort=0 velocity=100 -> lower=-0.001 upper=0.001 effort=0 velocity=1
- joint FR_tilt_joint: limit lower=-0.01 upper=-0.01 effort=0 velocity=100 -> lower=-0.001 upper=-0.001 effort=0 velocity=1
