Commit message: update

File: resources/robots/go1/urdf/go1.urdf (robot description, URDF)
Before this commit: robot go1_description, 23 links, 22 joints
Links:
- link FL_hip: geometry collision cylinder length=0.04 radius=0.046; visual mesh filename=../meshes/hip.stl scale=1 1 1
- link FR_hip: geometry collision cylinder length=0.04 radius=0.046; visual mesh filename=../meshes/hip.stl scale=1 1 1
- link RL_hip: geometry collision cylinder length=0.04 radius=0.046; visual mesh filename=../meshes/hip.stl scale=1 1 1
- link RR_hip: geometry collision cylinder length=0.04 radius=0.046; visual mesh filename=../meshes/hip.stl scale=1 1 1
